File: testCad/KeyboardTest2/KeyboardTest2.kicad_pcb (KiCad board)
At the start: 2 copper layers, 131.5 x 84 mm, 44 parts, among them J1 Conn_02x12_Top_Bottom, J2 AudioJack4

Commit message: 3D cad and pcb layout
Parts:
- J1: moved to B.Cu
- turned J1 to 180 degrees
Connections:
- J1 pad 10: M3OUT -> COL4
- J1 pad 11: M2OUT -> COL5
- J1 pad 12: M1OUT -> ROW1
- J1 pad 13: unconnected-(J1-Pin_13-Pad13) -> Net-(J1-Pin_13)
- J1 pad 14: unconnected-(J1-Pin_14-Pad14) -> Net-(J1-Pin_14)
- J1 pad 16: MIN -> unconnected-(J1-Pin_16-Pad16)
- J1 pad 17: ROW0 -> Net-(J1-Pin_17)
- J1 pad 18: COL0 -> Net-(J1-Pin_18)
- J1 pad 19: COL1 -> unconnected-(J1-Pin_19-Pad19)
- J1 pad 20: COL2 -> unconnected-(J1-Pin_20-Pad20)
- J1 pad 21: COL3 -> ROW2
- J1 pad 22: COL4 -> M3OUT
- J1 pad 23: COL5 -> M2OUT
- J1 pad 24: ROW1 -> M1OUT
- J1 pad 4: unconnected-(J1-Pin_4-Pad4) -> MIN
- J1 pad 5: Net-(J1-Pin_5) -> ROW0
- J1 pad 6: Net-(J1-Pin_6) -> COL0
- J1 pad 7: Net-(J1-Pin_7) -> COL1
- J1 pad 8: Net-(J1-Pin_8) -> COL2
- J1 pad 9: ROW2 -> COL3
- J2 pad R1: Net-(J1-Pin_7) -> Net-(J1-Pin_18)
- J2 pad R2: Net-(J1-Pin_8) -> Net-(J1-Pin_17)
- J2 pad S: Net-(J1-Pin_5) -> Net-(J1-Pin_14)
- J2 pad T: Net-(J1-Pin_6) -> Net-(J1-Pin_13)
Routing:
- net Net-(J1-Pin_13): track 0.00 -> 49.5 mm, vias 0 -> 1
- net Net-(J1-Pin_14): track 0.00 -> 42.4 mm, vias 0 -> 2
- net Net-(J1-Pin_17): track 0.00 -> 32.9 mm, vias 0 -> 1
- net Net-(J1-Pin_18): track 0.00 -> 31.8 mm, vias 0 -> 2
- added copper zone on B.Cu, net (none)
- added copper zone on F.Cu, net (none)
Other:
- outline, holes or cut-outs redrawn
