File: testCad/KeyboardTest2/KeyboardTest2_right.kicad_pcb (KiCad board)
At the start: 2 copper layers, 131.5 x 84 mm, 44 parts, among them J1 AudioJack4, J2 Conn_02x12_Top_Bottom

Commit message: 3D cad and pcb layout
Other:
- board size 131.5 x 84 mm -> 131.5 x 84.8 mm
